File: kb-split/kb-split.sch (KiCad schematic (older format))
At the start: 88 parts, among them J1 Conn_01x03_Male, SW1 SW_PUSH, SW10 SW_PUSH, SW11 SW_PUSH, SW12 SW_PUSH, SW13 SW_PUSH, SW14 SW_PUSH, SW15 SW_PUSH, SW16 SW_PUSH, SW17 SW_PUSH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

Commit message: Added Layout Template
Parts:
- added H1, H2: MountingHole_Pad, Mounting_Wuerth:Mounting_Wuerth_WA-SMSI-M1.6_H4.5mm_ThreadDepth2mm_97730456332, symbol Mechanical:MountingHole_Pad
- added J2: USB_C_Receptacle_USB2.0, Connector_USB:USB_C_Receptacle_HRO_TYPE-C-31-M-12, symbol Connector:USB_C_Receptacle_USB2.0
Connections:
- net LED: now also U1.24 (B0); no longer U1.1 (TX0/PD3)
- net SERIAL: now also U1.2 (RX1/PD2); no longer U1.6 (3/PD0)
- net at LED7.2 (DOUT): now also LED8.4 (DIN)
- new net: J2.A1 (GND), J2.A12 (GND), J2.B1 (GND), J2.B12 (GND)
- new net: J2.A4 (VBUS), J2.A9 (VBUS), J2.B4 (VBUS), J2.B9 (VBUS)
- new net: H1.1, J2.A7 (D-)
- new net: H2.1, J2.B6 (D+)
Other:
- moved on the sheet: J1, RSW1
Changed lines of the file:
@@
 	7950 6750 8200 6750
-Wire Wire Line
-	8850 6750 9050 6750
 Wire Wire Line
 	9650 6750 9900 6750
@@
 Text GLabel 1750 2450 0    50   Input ~ 0
 ROW0
-Text GLabel 1750 1850 0    50   Input ~ 0
+Text GLabel 3150 1850 2    50   Input ~ 0
 LED
 Text GLabel 1750 2550 0    50   Input ~ 0
@@
 L kbd:SW_PUSH RSW1
 U 1 1 60850878
-P 2000 4400
-F 0 "RSW1" H 2000 4655 50  0000 C CNN
-F 1 "SW_PUSH" H 2000 4564 50  0000 C CNN
-F 2 "kbd:CherryMX_Hotswap" H 2000 4400 50  0001 C CNN
-F 3 "" H 2000 4400 50  0000 C CNN
-	1    2000 4400
+P 2500 4000
+F 0 "RSW1" H 2500 4255 50  0000 C CNN
+F 1 "SW_PUSH" H 2500 4164 50  0000 C CNN
+F 2 "kbd:CherryMX_Hotswap" H 2500 4000 50  0001 C CNN
+F 3 "" H 2500 4000 50  0000 C CNN
+	1    2500 4000
 	1    0    0    -1
 $EndComp
@@
 L power:GND #PWR0104
 U 1 1 60852B2A
-P 2300 4400
-F 0 "#PWR0104" H 2300 4150 50  0001 C CNN
-F 1 "GND" H 2305 4227 50  0000 C CNN
-F 2 "" H 2300 4400 50  0001 C CNN
-F 3 "" H 2300 4400 50  0001 C CNN
-	1    2300 4400
-	1    0    0    -1
-$EndComp
-Text GLabel 1700 4400 0    50   Input ~ 0
+P 2800 4000
+F 0 "#PWR0104" H 2800 3750 50  0001 C CNN
+F 1 "GND" H 2805 3827 50  0000 C CNN
+F 2 "" H 2800 4000 50  0001 C CNN
+F 3 "" H 2800 4000 50  0001 C CNN
+	1    2800 4000
+	1    0    0    -1
+$EndComp
+Text GLabel 2200 4000 0    50   Input ~ 0
 RESET
 $Comp
 L Connector:Conn_01x03_Male J1
 U 1 1 6088D94E
-P 1700 5250
-F 0 "J1" H 1808 5531 50  0000 C CNN
-F 1 "Conn_01x03_Male" H 1808 5440 50  0000 C CNN
-F 2 "Connector_PinHeader_1.00mm:PinHeader_1x03_P1.00mm_Horizontal" H 1700 5250 50  0001 C CNN
-F 3 "~" H 1700 5250 50  0001 C CNN
-	1    1700 5250
+P 2100 4750
+F 0 "J1" H 2208 5031 50  0000 C CNN
+F 1 "Conn_01x03_Male" H 2208 4940 50  0000 C CNN
+F 2 "Connector_PinHeader_1.00mm:PinHeader_1x03_P1.00mm_Horizontal" H 2100 4750 50  0001 C CNN
+F 3 "~" H 2100 4750 50  0001 C CNN
+	1    2100 4750
 	1    0    0    -1
 $EndComp
@@
 L power:GND #PWR0105
 U 1 1 608B623C
-P 1900 5350
-F 0 "#PWR0105" H 1900 5100 50  0001 C CNN
-F 1 "GND" H 1905 5177 50  0000 C CNN
-F 2 "" H 1900 5350 50  0001 C CNN
-F 3 "" H 1900 5350 50  0001 C CNN
-	1    1900 5350
+P 2300 4850
+F 0 "#PWR0105" H 2300 4600 50  0001 C CNN
+F 1 "GND" H 2305 4677 50  0000 C CNN
+F 2 "" H 2300 4850 50  0001 C CNN
+F 3 "" H 2300 4850 50  0001 C CNN
+	1    2300 4850
 	1    0    0    -1
 $EndComp
@@
 L power:VCC #PWR0106
 U 1 1 608B7084
-P 2500 5250
-F 0 "#PWR0106" H 2500 5100 50  0001 C CNN
-F 1 "VCC" H 2515 5423 50  0000 C CNN
-F 2 "" H 2500 5250 50  0001 C CNN
-F 3 "" H 2500 5250 50  0001 C CNN
-	1    2500 5250
-	1    0    0    -1
-$EndComp
-Text GLabel 2000 5150 2    50   Input ~ 0
+P 2900 4750
+F 0 "#PWR0106" H 2900 4600 50  0001 C CNN
+F 1 "VCC" H 2915 4923 50  0000 C CNN
+F 2 "" H 2900 4750 50  0001 C CNN
+F 3 "" H 2900 4750 50  0001 C CNN
+	1    2900 4750
+	1    0    0    -1
+$EndComp
+Text GLabel 2400 4650 2    50   Input ~ 0
 SERIAL
-Text GLabel 1750 2350 0    50   Input ~ 0
+Text GLabel 1750 1950 0    50   Input ~ 0
 SERIAL
 Wire Wire Line
-	1900 5250 2500 5250
-Wire Wire Line
-	2000 5150 1900 5150
+	2300 4750 2900 4750
+Wire Wire Line
+	2400 4650 2300 4650
+Wire Wire Line
+	8800 6750 9050 6750
+$Comp
+L Connector:USB_C_Receptacle_USB2.0 J2
+U 1 1 60997110
+P 4200 6500
+F 0 "J2" H 4307 7367 50  0000 C CNN
+F 1 "USB_C_Receptacle_USB2.0" H 4307 7276 50  0000 C CNN
+F 2 "Connector_USB:USB_C_Receptacle_HRO_TYPE-C-31-M-12" H 4350 6500 50  0001 C CNN
+F 3 "https://www.usb.org/sites/default/files/documents/usb_type-c.zip" H 4350 6500 50  0001 C CNN
+	1    4200 6500
+	1    0    0    -1
+$EndComp
+$Comp
+L Mechanical:MountingHole_Pad H1
+U 1 1 609DC973
+P 5350 6050
+F 0 "H1" H 5450 6099 50  0000 L CNN
+F 1 "MountingHole_Pad" H 5450 6008 50  0000 L CNN
+F 2 "Mounting_Wuerth:Mounting_Wuerth_WA-SMSI-M1.6_H4.5mm_ThreadDepth2mm_97730456332" H 5350 6050 50  0001 C CNN
+F 3 "~" H 5350 6050 50  0001 C CNN
+	1    5350 6050
+	1    0    0    -1
+$EndComp
+Wire Wire Line
+	4800 6400 5350 6400
+Wire Wire Line
+	5350 6400 5350 6150
+$Comp
+L Mechanical:MountingHole_Pad H2
+U 1 1 609ED140
+P 5300 6850
+F 0 "H2" H 5400 6899 50  0000 L CNN
+F 1 "MountingHole_Pad" H 5400 6808 50  0000 L CNN
+F 2 "Mounting_Wuerth:Mounting_Wuerth_WA-SMSI-M1.6_H4.5mm_ThreadDepth2mm_97730456332" H 5300 6850 50  0001 C CNN
+F 3 "~" H 5300 6850 50  0001 C CNN
+	1    5300 6850
+	1    0    0    -1
+$EndComp
+Wire Wire Line
+	5000 6950 5000 6700
+Wire Wire Line
+	5000 6700 4800 6700
+Wire Wire Line
+	5000 6950 5300 6950
 $EndSCHEMATC
