File: kb-split/kb-split.sch (KiCad schematic (older format))
At the start: 137 parts, among them J1 Conn_01x03_Male, J2 USB_C_Receptacle_USB2.0, SW1 SW_PUSH, SW10 SW_PUSH, SW11 SW_PUSH, SW12 SW_PUSH, SW13 SW_PUSH, SW14 SW_PUSH, SW15 SW_PUSH, SW16 SW_PUSH, SW17 SW_PUSH, SW18 SW_PUSH, SW19 SW_PUSH, SW2 SW_PUSH, SW20 SW_PUSH, SW21 Rotary_Encoder_Switch, SW22 SW_PUSH, SW23 SW_PUSH, SW24 SW_PUSH, SW25 SW_PUSH, SW26 SW_PUSH, SW27 SW_PUSH, SW28 SW_PUSH, SW3 SW_PUSH, SW4 SW_PUSH, SW5 SW_PUSH, SW6 SW_PUSH, SW7 SW_PUSH, SW8 SW_PUSH, SW9 SW_PUSH, U1 SRV05-4, U2 ATmega32U4-AU, Y1 Crystal_GND24_Small

Commit message: Create reversible Cystal footprint
Parts:
- C1, C10, C11, C12, C13, C14, C15, C16, C17, C18, C19, C2, C20, C21, C22, C23, C24, C25, C26, C27, C28, C29, C3, C30, C31, C32, C33, C34, C35, C36, C37, C38, C4, C5, C6, C7, C8, C9: footprint Capacitor_SMD:C_0805_2012Metric -> reversible-kicad-footprints:C-0805_2012Metric
- D1, D10, D11, D12, D13, D14, D15, D16, D17, D18, D19, D2, D20, D21, D22, D23, D24, D25, D26, D27, D3, D4, D5, D6, D7, D8, D9: footprint Diode_SMD:D_SOD-123 -> reversible-kicad-footprints:D_SOD-123
- F1: footprint Fuse:Fuse_1206_3216Metric -> reversible-kicad-footprints:Fuse_1206_3216Metric
- J2: footprint Connector_USB:USB_C_Receptacle_HRO_TYPE-C-31-M-12 -> reversible-kicad-footprints:HRO-TYPE-C-31-M-12-HandSoldering-NoSBU; symbol Connector:USB_C_Receptacle_USB2.0 -> reversible-kicad-symbols:HRO-TYPE-C-31-M-12-HandSoldering-NoSBU
- LED1, LED2, LED3, LED4: footprint kbd:YS-SK6812MINI-E -> reversible-kicad-footprints:SK6812Mini-E
- LED10, LED11, LED12, LED13, LED14, LED15, LED16, LED17, LED18, LED19, LED20, LED21, LED22, LED23, LED24, LED25, LED26, LED27, LED28, LED29, LED30, LED31, LED5, LED6, LED7, LED8, LED9: footprint kbd:YS-SK6812MINI-E -> reversible-kicad-footprints:MX-1U-SK6812Mini-E
- R1, R2, R3, R4, R5, R6: footprint Resistor_SMD:R_0805_2012Metric -> reversible-kicad-footprints:R-0805_2012Metric
- SW1, SW10, SW11, SW12, SW13, SW14, SW15, SW16, SW17, SW18, SW19, SW2, SW20, SW22, SW23, SW24, SW25, SW26, SW27, SW3, SW4, SW5, SW6, SW7, SW8, SW9: footprint kbd:CherryMX_Hotswap -> reversible-kicad-footprints:MX-1U-Hotswap
- SW21: footprint Keebio-Parts:RotaryEncoder_Alps_EC11E-Switch_Vertical_H20mm -> reversible-kicad-footprints:MX-1U-EC11_Switch
- SW28: footprint random-keyboard-parts:SKQG-1155865 -> reversible-kicad-footprints:SMD_Push
- U1: footprint Package_TO_SOT_SMD:SOT-23-6 -> reversible-kicad-footprints:SOT-23-6
- Y1: footprint Crystal:Crystal_SMD_3225-4Pin_3.2x2.5mm_HandSoldering -> intositeme:Reversible-Crystal_SMD_3225-4pin_3.2x2.5mm
Connections:
- wire segments 279 -> 378
Other:
- moved on the sheet: C10, C11, C12, C13, C14, C15, C16, C17, C18, C19, C20, C21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

Commit message: Layout components
Parts:
- removed C10, C12, C13, C15, C17, C19, C20, C22, C24, C26, C27, C29, C31, C33, C35, C37, C8: 0.1uF, reversible-kicad-footprints:C-0805_2012Metric, symbol Device:C_Small
- added H1, H2, H3, H4, H5: MountingHole, kbd:M2_HOLE_v3, symbol Mechanical:MountingHole
- LED25: footprint reversible-kicad-footprints:MX-1U-SK6812Mini-E -> reversible-kicad-footprints:SK6812Mini-E
- renumbered C16 to C10, C18 to C11, C21 to C12, C23 to C13, C25 to C14, C7 to C15, C28 to C16, C30 to C17, C32 to C18, C34 to C19, C36 to C20, C38 to C21, C9 to C7, C11 to C8, C14 to C9, J2 to J1, J1 to J2, SW21 to SW15, SW15 to SW16, SW16 to SW17, SW17 to SW18, SW18 to SW19, SW19 to SW20, SW20 to SW21, SW28 to SW22, SW22 to SW23, SW23 to SW24, SW24 to SW25, SW25 to SW26, SW26 to SW27, SW27 to SW28

Commit message: Done routing.
Parts:
- removed C20, C21: 0.1uF, reversible-kicad-footprints:C-0805_2012Metric, symbol Device:C_Small
Connections:
- net MISO is gone; now on net COL0: ISP1.1 (Pin_1), U2.11 (PB3)
- net MOSI is gone; now on net COL1: ISP1.4 (Pin_4), U2.10 (PB2)
- net SCK is gone; now on net COL2: ISP1.3 (Pin_3), U2.9 (PB1)
- net +5V: now also J2.2 (Pin_2)
- net COL0: no longer U2.38 (PF5)
- net COL1: no longer U2.37 (PF6)
- net COL2: no longer U2.36 (PF7)
- net COL3: now also U2.8 (PB0); no longer U2.32 (PC7)
- net COL4: now also U2.41 (PF0); no longer U2.31 (PC6)
- net COL5: now also SW13.1, SW21.1, SW28.1, SW6.1, U2.38 (PF5); no longer U2.30 (PB6)
- net COL6: now also SW14.1, SW15.S2, SW7.1, U2.27 (PD7); no longer U2.29 (PB5)
- net ENC0: now also U2.40 (PF1); no longer U2.18 (PD0)
- net ENC1: now also U2.39 (PF4); no longer U2.19 (PD1)
- net GND: now also C7.1, C8.1, LED4.3 (VSS); no longer C7.2, C8.2, LED3.3 (VSS), LED4.1 (VDD)
- net LED: now also LED31.4 (DIN), U2.42 (AREF); no longer LED4.4 (DIN), U2.22 (PD5)
- net ROW0: now also U2.26 (PD6); no longer U2.28 (PB4)
- net ROW1: now also U2.28 (PB4); no longer U2.27 (PD7)
- net ROW2: now also U2.29 (PB5); no longer U2.26 (PD6)
- net VCC: now also C7.2, C8.2, ISP1.2 (Pin_2), LED4.1 (VDD); no longer C7.1, C8.1, J2.2 (Pin_2), LED4.3 (VSS)
- net at LED4.2 (DOUT): now also LED17.4 (DIN); no longer LED3.4 (DIN)
- net at LED3.2 (DOUT): now also LED15.4 (DIN); no longer LED2.4 (DIN)
- net at LED2.2 (DOUT): now also LED28.4 (DIN); no longer LED1.4 (DIN)
- net at LED1.2 (DOUT): now also LED20.4 (DIN); no longer LED5.4 (DIN)
- net at LED11.2 (DOUT): no longer LED18.4 (DIN)
- net at LED18.2 (DOUT): now also LED4.4 (DIN); no longer LED17.4 (DIN)
- net at LED16.2 (DOUT): now also LED3.4 (DIN); no longer LED15.4 (DIN)
- net at LED12.2 (DOUT): now also LED5.4 (DIN); no longer LED19.4 (DIN)
- net at LED19.2 (DOUT): now also LED1.4 (DIN); no longer LED20.4 (DIN)
- net at LED25.2 (DOUT): now also LED18.4 (DIN); no longer LED31.4 (DIN)
- net at LED29.2 (DOUT): now also LED2.4 (DIN); no longer LED28.4 (DIN)
- net at LED26.2 (DOUT): now also LED19.4 (DIN)
- no-connect marks 14 -> 13
Other:
- moved on the sheet: C10, C11, C12, C13, C14, C16, C17, C18, C19, C7, C8, C9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

Commit message: Added trs and fix gerbers export
Parts:
- added J3: AudioPlug3, reversible-kicad-footprints:PJ-3136-B, symbol Connector:AudioPlug3
- J1: symbol reversible-kicad-symbols:HRO-TYPE-C-31-M-12-HandSoldering-NoSBU -> kb-split-rescue:HRO-TYPE-C-31-M-12-HandSoldering-NoSBU-reversible-kicad-symbols
- SW22: symbol kbd:SW_PUSH -> kb-split-rescue:SW_PUSH-kbd
Connections:
- net +5V: now also J3.R
- net GND: now also J3.T
- net SERIAL: now also J3.S
Changed lines of the file:
@@
 RESET
 $Comp
-L kbd:SW_PUSH SW22
+L kb-split-rescue:SW_PUSH-kbd SW22
 U 1 1 60820895
 P 1600 3400
@@
 	2250 1750 2150 1750
 $Comp
-L reversible-kicad-symbols:HRO-TYPE-C-31-M-12-HandSoldering-NoSBU J1
+L kb-split-rescue:HRO-TYPE-C-31-M-12-HandSoldering-NoSBU-reversible-kicad-symbols J1
 U 1 1 60997110
 P 1400 1750
@@
 NoConn ~ 3650 7650
 NoConn ~ 3650 7550
+Text GLabel 4600 5150 2    50   Input ~ 0
+SERIAL
+$Comp
+L power:+5V #PWR0103
+U 1 1 600DB243
+P 5000 5250
+F 0 "#PWR0103" H 5000 5100 50  0001 C CNN
+F 1 "+5V" H 5015 5423 50  0000 C CNN
+F 2 "" H 5000 5250 50  0001 C CNN
+F 3 "" H 5000 5250 50  0001 C CNN
+	1    5000 5250
+	1    0    0    -1
+$EndComp
+$Comp
+L power:GND #PWR0104
+U 1 1 600DBDBB
+P 4600 5350
+F 0 "#PWR0104" H 4600 5100 50  0001 C CNN
+F 1 "GND" H 4605 5177 50  0000 C CNN
+F 2 "" H 4600 5350 50  0001 C CNN
+F 3 "" H 4600 5350 50  0001 C CNN
+	1    4600 5350
+	1    0    0    -1
+$EndComp
+$Comp
+L Connector:AudioPlug3 J3
+U 1 1 600BE536
+P 4000 5250
+F 0 "J3" H 4057 5617 50  0000 C CNN
+F 1 "AudioPlug3" H 4057 5526 50  0000 C CNN
+F 2 "reversible-kicad-footprints:PJ-3136-B" H 4100 5200 50  0001 C CNN
+F 3 "~" H 4100 5200 50  0001 C CNN
+	1    4000 5250
+	1    0    0    -1
+$EndComp
+Wire Wire Line
+	4600 5250 5000 5250
 $EndSCHEMATC
