File: kb-split/kb-split-elite-c.sch (KiCad schematic (older format))
At the start: 137 parts, among them J1 Conn_01x03_Male, J2 USB_C_Receptacle_USB2.0, SW1 SW_PUSH, SW10 SW_PUSH, SW11 SW_PUSH, SW12 SW_PUSH, SW13 SW_PUSH, SW14 SW_PUSH, SW15 SW_PUSH, SW16 SW_PUSH, SW17 SW_PUSH, SW18 SW_PUSH, SW19 SW_PUSH, SW2 SW_PUSH, SW20 SW_PUSH, SW21 Rotary_Encoder_Switch, SW22 SW_PUSH, SW23 SW_PUSH, SW24 SW_PUSH, SW25 SW_PUSH, SW26 SW_PUSH, SW27 SW_PUSH, SW28 SW_PUSH, SW3 SW_PUSH, SW4 SW_PUSH, SW5 SW_PUSH, SW6 SW_PUSH, SW7 SW_PUSH, SW8 SW_PUSH, SW9 SW_PUSH, U1 SRV05-4, U2 ATmega32U4-AU, Y1 Crystal_GND24_Small

Commit message: redo schematic to remove eliteC and use atmega32u4 directly
Parts:
- removed C10, C11, C12, C13, C14, C15, C16, C17, C18, C19, C20, C21, C22, C23, C24, C25, C26, C27, C28, C29, C30, C31, C32, C33, C34, C35, C36, C37, C38, C8, C9: 0.1uF, Capacitor_SMD:C_0805_2012Metric, symbol Device:C_Small
- removed ISP1: Conn_02x03, Connector_PinSocket_2.54mm:PinSocket_2x03_P2.54mm_Vertical, symbol Connector_Generic:Conn_02x03_Odd_Even
- removed U1: SRV05-4, Package_TO_SOT_SMD:SOT-23-6, symbol Power_Protection:SRV05-4
- added ISP: Conn_02x03, symbol Connector_Generic_MountingPin:Conn_02x03_Odd_Even_MountingPin
- added RSW1: SW_PUSH, kbd:CherryMX_Hotswap, symbol kb-split-rescue:SW_PUSH-kbd
- added U1: Elite-C, Keebio-Parts:Elite-C-castellated-29pin-holes, symbol kb-split-rescue:Elite-C-keebio
- C?: renamed from C7; footprint Capacitor_SMD:C_0805_2012Metric -> (none)
- C?: renamed from C3; footprint Capacitor_SMD:C_0805_2012Metric -> (none)
- C?: renamed from C4; footprint Capacitor_SMD:C_0805_2012Metric -> (none)
- C?: renamed from C5; footprint Capacitor_SMD:C_0805_2012Metric -> (none)
- C?: renamed from C6; footprint Capacitor_SMD:C_0805_2012Metric -> (none)
- C?: renamed from C1; footprint Capacitor_SMD:C_0805_2012Metric -> (none)
- C?: renamed from C2; footprint Capacitor_SMD:C_0805_2012Metric -> (none)
- D1, D10, D11, D12, D13, D14, D15, D16, D17, D18, D19, D2, D20, D21, D22, D23, D24, D25, D26, D27, D3, D4, D5, D6, D7, D8, D9: footprint Diode_SMD:D_SOD-123 -> Diode_SMD:D_SOD-323
- F?: renamed from F1; footprint Fuse:Fuse_1206_3216Metric -> (none)
- J1: footprint Connector_PinSocket_2.54mm:PinSocket_1x03_P2.54mm_Horizontal -> Connector_PinHeader_1.00mm:PinHeader_1x03_P1.00mm_Horizontal
- R?: renamed from R6; footprint Resistor_SMD:R_0805_2012Metric -> (none)
- R?: renamed from R4; footprint Resistor_SMD:R_0805_2012Metric -> (none)
- R?: renamed from R5; footprint Resistor_SMD:R_0805_2012Metric -> (none)
- R?: renamed from R1; footprint Resistor_SMD:R_0805_2012Metric -> (none)
- R?: renamed from R2; footprint Resistor_SMD:R_0805_2012Metric -> (none)
- R?: renamed from R3; footprint Resistor_SMD:R_0805_2012Metric -> (none)
- SW?: renamed from SW28; footprint random-keyboard-parts:SKQG-1155865 -> (none)
- Y?: renamed from Y1; footprint Crystal:Crystal_SMD_3225-4Pin_3.2x2.5mm_HandSoldering -> (none)
Connections:
- net COL0: now also U1.20 (A3/PF4)
- net COL1: now also U1.19 (A2/PF5)
- net COL2: now also U1.18 (A1/PF6)
- net COL3: now also U1.17 (A0/PF7)
- net COL4: now also U1.16 (15/PB1)
- net COL5: now also U1.15 (14/PB3)
- net COL6: now also U1.14 (16/PB2)
- net ENC0: now also U1.11 (8/PB4)
- net ENC1: now also U1.12 (9/PB5)
- net GND: now also ISP.6 (Pin_6), RSW1.2, U1.23 (GND)
- net LED: now also U1.24 (B0)
- net MISO: now also ISP.1 (Pin_1)
- net MOSI: now also ISP.4 (Pin_4)
- net RESET: now also ISP.5 (Pin_5), RSW1.1, U1.22 (RST)
- net ROW0: now also U1.7 (4/PD4)
- net ROW1: now also U1.8 (5/PC6)
- net ROW2: now also U1.9 (6/PD7)
- net ROW3: now also U1.10 (7/PE6)
- net SCK: now also ISP.3 (Pin_3)
- net SERIAL: now also U1.2 (RX1/PD2)
- net VCC: now also LED1.1 (VDD), LED10.1 (VDD), LED11.1 (VDD), LED12.1 (VDD), LED13.1 (VDD), LED14.1 (VDD), LED15.1 (VDD), LED16.1 (VDD), LED17.1 (VDD), LED18.1 (VDD), LED19.1 (VDD), LED2.1 (VDD), LED20.1 (VDD), LED21.1 (VDD), LED22.1 (VDD), LED23.1 (VDD), LED24.1 (VDD), LED25.1 (VDD), LED26.1 (VDD), LED27.1 (VDD), LED28.1 (VDD), LED29.1 (VDD), LED3.1 (VDD), LED30.1 (VDD), LED31.1 (VDD), LED4.1 (VDD), LED5.1 (VDD), LED6.1 (VDD), LED7.1 (VDD), LED8.1 (VDD), LED9.1 (VDD), ISP.2 (Pin_2), U1.21 (VCC)
- no-connect marks 14 -> 11
