File: kb-split/kb-split.kicad_pcb (KiCad board)
At the start: 2 copper layers, 3.6 x 3.1 mm, 88 parts, among them J1 Conn_01x03_Male, SW1 SW_PUSH, SW10 SW_PUSH, SW11 SW_PUSH, SW12 SW_PUSH, SW13 SW_PUSH, SW14 SW_PUSH, SW15 SW_PUSH, SW16 SW_PUSH, SW17 SW_PUSH, SW18 SW_PUSH, SW19 SW_PUSH, SW2 SW_PUSH, SW20 SW_PUSH, SW21 Rotary_Encoder_Switch, SW22 SW_PUSH, SW23 SW_PUSH, SW24 SW_PUSH, SW25 SW_PUSH, SW26 SW_PUSH, SW27 SW_PUSH, SW3 SW_PUSH, SW4 SW_PUSH, SW5 SW_PUSH, SW6 SW_PUSH, SW7 SW_PUSH, SW8 SW_PUSH, SW9 SW_PUSH, U1 Elite-C

Commit message: Added Layout Template
Parts:
- added H1: MountingHole_Pad, Mounting_Wuerth:Mounting_Wuerth_WA-SMSI-M1.6_H4.5mm_ThreadDepth2mm_97730456332, B.Cu at (65.0, 69.1)
- added H2: MountingHole_Pad, Mounting_Wuerth:Mounting_Wuerth_WA-SMSI-M1.6_H4.5mm_ThreadDepth2mm_97730456332, B.Cu at (56.6, 69.3)
- added J2: USB_C_Receptacle_USB2.0, Connector_USB:USB_C_Receptacle_HRO_TYPE-C-31-M-12, B.Cu at (61.0, 89.4)
- added REF**: Layout, intositeme:Layout, F.Cu at (133.3, 23.8)
- LED5, SW21: moved to B.Cu
- moved D1 351.9 mm to (134.6, 30.5), turned to 270 degrees
- moved SW8 284.2 mm to (142.9, 52.4), turned to 180 degrees
- moved LED5 267.8 mm to (143.0, 27.9)
- moved SW10 265.8 mm to (181.0, 52.4), turned to 180 degrees
- moved SW9 263.3 mm to (161.9, 52.4), turned to 180 degrees
- moved SW5 249.3 mm to (219.1, 33.3), turned to 180 degrees
- moved SW6 241.4 mm to (238.1, 33.3), turned to 180 degrees
- moved SW15 236.5 mm to (142.9, 71.4), turned to 180 degrees
- moved U1 234.6 mm to (278.9, 84.1), turned to 240 degrees
- moved SW16 223.8 mm to (161.9, 71.4), turned to 180 degrees
- moved SW11 220.8 mm to (200.0, 52.4), turned to 180 degrees
- moved SW17 214.1 mm to (181.0, 71.4), turned to 180 degrees
- moved SW23 213.5 mm to (161.9, 90.5), turned to 180 degrees
- moved SW12 209.4 mm to (219.1, 52.4), turned to 180 degrees
- moved SW22 208.9 mm to (142.9, 90.5), turned to 180 degrees
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Connections:
- LED8 pad 4: Net-(LED8-Pad4) -> Net-(LED7-Pad2)
- U1 pad 1: LED -> Net-(U1-Pad1)
- U1 pad 2: Net-(U1-Pad2) -> SERIAL
- U1 pad 24: Net-(U1-Pad24) -> LED
- U1 pad 6: SERIAL -> Net-(U1-Pad6)
Routing:
- net Net-(H2-Pad1): track 0.00 -> 17.3 mm
- net Net-(H1-Pad1): track 0.00 -> 16.8 mm

Commit message: redo schematic to remove eliteC and use atmega32u4 directly
Parts:
- removed H1, H2: MountingHole_Pad, Mounting_Wuerth:Mounting_Wuerth_WA-SMSI-M1.6_H4.5mm_ThreadDepth2mm_97730456332
- removed RSW1: SW_PUSH, kbd:CherryMX_Hotswap
- added C1: 22pF, Capacitor_SMD:C_0805_2012Metric, F.Cu at (448.3, 118.1)
- added C10: 0.1uF, Capacitor_SMD:C_0805_2012Metric, F.Cu at (454.1, 116.6)
- added C11: 0.1uF, Capacitor_SMD:C_0805_2012Metric, F.Cu at (503.4, 67.2)
- added C12: 0.1uF, Capacitor_SMD:C_0805_2012Metric, B.Cu at (101.6, 52.4)
- added C13: 0.1uF, Capacitor_SMD:C_0805_2012Metric, B.Cu at (120.7, 52.4)
- added C14: 0.1uF, Capacitor_SMD:C_0805_2012Metric, B.Cu at (139.7, 52.4)
- added C15: 0.1uF, Capacitor_SMD:C_0805_2012Metric, F.Cu at (483.2, 86.3)
- added C16: 0.1uF, Capacitor_SMD:C_0805_2012Metric, F.Cu at (442.4, 128.2)
- added C17: 0.1uF, Capacitor_SMD:C_0805_2012Metric, F.Cu at (469.3, 101.7)
- added C18: 0.1uF, Capacitor_SMD:C_0805_2012Metric, F.Cu at (466.1, 106.5)
- added C19: 0.1uF, Capacitor_SMD:C_0805_2012Metric, F.Cu at (460.4, 109.9)
- added C2: 22pF, Capacitor_SMD:C_0805_2012Metric, F.Cu at (436.8, 116.2)
- added C20: 0.1uF, Capacitor_SMD:C_0805_2012Metric, F.Cu at (448.3, 121.5)
- added C21: 0.1uF, Capacitor_SMD:C_0805_2012Metric, F.Cu at (469.3, 98.3)
- added C22: 0.1uF, Capacitor_SMD:C_0805_2012Metric, F.Cu at (442.4, 124.8)
- added C23: 0.1uF, Capacitor_SMD:C_0805_2012Metric, F.Cu at (486.4, 82.9)
- added C24: 0.1uF, Capacitor_SMD:C_0805_2012Metric, F.Cu at (489.6, 79.6)
- added C25: 0.1uF, Capacitor_SMD:C_0805_2012Metric, F.Cu at (497.6, 71.4)
- added C26: 0.1uF, Capacitor_SMD:C_0805_2012Metric, F.Cu at (477.4, 91.6)
- added C27: 0.1uF, Capacitor_SMD:C_0805_2012Metric, F.Cu at (434.5, 133.0)
- added C28: 0.1uF, Capacitor_SMD:C_0805_2012Metric, F.Cu at (451.5, 113.3)
- added C29: 0.1uF, Capacitor_SMD:C_0805_2012Metric, F.Cu at (463.6, 103.1)
- added C3: 0.1uF, Capacitor_SMD:C_0805_2012Metric, F.Cu at (436.7, 129.6)
- added C30: 0.1uF, Capacitor_SMD:C_0805_2012Metric, F.Cu at (477.4, 88.3)
- added C31: 0.1uF, Capacitor_SMD:C_0805_2012Metric, F.Cu at (460.4, 106.6)
- added C32: 0.1uF, Capacitor_SMD:C_0805_2012Metric, F.Cu at (500.8, 63.8)
- added C33: 0.1uF, Capacitor_SMD:C_0805_2012Metric, F.Cu at (500.8, 60.5)
- added C34: 0.1uF, Capacitor_SMD:C_0805_2012Metric, F.Cu at (454.6, 109.9)
- added C35: 0.1uF, Capacitor_SMD:C_0805_2012Metric, F.Cu at (442.6, 121.5)
- added C36: 0.1uF, Capacitor_SMD:C_0805_2012Metric, F.Cu at (442.6, 118.1)
- added C37: 0.1uF, Capacitor_SMD:C_0805_2012Metric, F.Cu at (436.7, 126.3)
- added C38: 0.1uF, Capacitor_SMD:C_0805_2012Metric, F.Cu at (483.9, 79.6)
- added C4: 0.1uF, Capacitor_SMD:C_0805_2012Metric, F.Cu at (480.6, 82.9)
- added C5: 0.1uF, Capacitor_SMD:C_0805_2012Metric, F.Cu at (489.6, 76.2)
- added C6: 10uF, Capacitor_SMD:C_0805_2012Metric, F.Cu at (497.6, 68.1)
- added C7: 1uF, Capacitor_SMD:C_0805_2012Metric, F.Cu at (471.7, 95.0)
- added C8: 0.1uF, Capacitor_SMD:C_0805_2012Metric, F.Cu at (483.2, 89.6)
- added C9: 0.1uF, Capacitor_SMD:C_0805_2012Metric, F.Cu at (440.2, 133.0)
- added F1: Polyfuse_Small, Fuse:Fuse_1206_3216Metric, F.Cu at (448.1, 124.8)
- added ISP1: Conn_02x03, Connector_PinSocket_2.54mm:PinSocket_2x03_P2.54mm_Vertical, F.Cu at (403.9, 170.2)
- added R1: 5.1k, Resistor_SMD:R_0805_2012Metric, F.Cu at (404.4, 136.2)
- added R2: 5.1k, Resistor_SMD:R_0805_2012Metric, F.Cu at (399.9, 136.3)
- added R3: 10k, Resistor_SMD:R_0805_2012Metric, F.Cu at (395.5, 136.3)
- added R4: 22, Resistor_SMD:R_0805_2012Metric, F.Cu at (362.5, 136.2)
- added R5: 22, Resistor_SMD:R_0805_2012Metric, F.Cu at (358.1, 136.2)
- added R6: 10k, Resistor_SMD:R_0805_2012Metric, F.Cu at (353.7, 136.2)
- added SW28: SW_PUSH, random-keyboard-parts:SKQG-1155865, F.Cu at (370.7, 133.2)
- added U2: ATmega32U4-AU, Package_QFP:TQFP-44_10x10mm_P0.8mm, F.Cu at (358.7, 127.5)
- added Y1: Crystal_GND24_Small, Crystal:Crystal_SMD_3225-4Pin_3.2x2.5mm_HandSoldering, F.Cu at (477.7, 77.0)
- D1, D2: footprint Diode_SMD:D_SOD-323 -> Diode_SMD:D_SOD-123; moved to B.Cu
- D10, D11, D12, D13, D14, D15, D16, D17, D18, D19, D20, D21, D22, D23, D24, D25, D26, D27, D3, D4, D5, D6, D7, D8, D9: footprint Diode_SMD:D_SOD-323 -> Diode_SMD:D_SOD-123
- J1: footprint Connector_PinHeader_1.00mm:PinHeader_1x03_P1.00mm_Horizontal -> Connector_PinSocket_2.54mm:PinSocket_1x03_P2.54mm_Horizontal
- J2, SW21: moved to F.Cu
- LED6, LED7: moved to B.Cu
- U1: value Elite-C -> SRV05-4; footprint Keebio-Parts:Elite-C-castellated-29pin-holes -> Package_TO_SOT_SMD:SOT-23-6; moved to F.Cu
- moved D2 349.8 mm to (118.3, 59.5), turned to 270 degrees
- moved J2 326.2 mm to (385.1, 126.1), turned to 0 degrees
- moved LED6 262.2 mm to (126.2, 54.8), turned to 180 degrees
- moved LED3 261.4 mm to (499.0, 51.5)
- moved LED7 254.8 mm to (145.3, 54.8), turned to 180 degrees
- moved D25 250.0 mm to (486.1, 66.2)
- moved LED8 243.0 mm to (487.7, 62.1)
- moved LED4 242.6 mm to (478.8, 71.7)
- moved D19 235.9 mm to (495.1, 61.4)
- moved D21 235.7 mm to (486.1, 69.5)
- moved LED13 233.3 mm to (499.0, 46.7)
- moved D23 225.1 mm to (474.9, 81.6)
- moved LED18 218.4 mm to (499.0, 41.9)
- moved D24 218.4 mm to (465.9, 86.4)
- moved D27 214.5 mm to (457.0, 96.0)
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Connections:
- J1 pad 2: VCC -> VBUS
- J2 pad A1: Net-(J2-PadA1) -> GND
- J2 pad A12: Net-(J2-PadA1) -> GND
- J2 pad A4: Net-(J2-PadA4) -> VBUS
- J2 pad A6: Net-(J2-PadA6) -> D+
- J2 pad A7: Net-(H1-Pad1) -> D-
- J2 pad A9: Net-(J2-PadA4) -> VBUS
- J2 pad B1: Net-(J2-PadA1) -> GND
- J2 pad B12: Net-(J2-PadA1) -> GND
- J2 pad B4: Net-(J2-PadA4) -> VBUS
- J2 pad B6: Net-(H2-Pad1) -> D+
- J2 pad B7: Net-(J2-PadB7) -> D-
- J2 pad B9: Net-(J2-PadA4) -> VBUS
- J2 pad S1: Net-(J2-PadS1) -> GND
- LED1 pad 1: VCC -> Net-(C8-Pad2)
- LED10 pad 1: VCC -> Net-(C16-Pad2)
- LED11 pad 1: VCC -> Net-(C17-Pad2)
- LED12 pad 1: VCC -> Net-(C19-Pad1)
- LED13 pad 1: VCC -> Net-(C19-Pad2)
- LED14 pad 1: VCC -> Net-(C20-Pad2)
- LED15 pad 1: VCC -> Net-(C21-Pad2)
- LED16 pad 1: VCC -> Net-(C22-Pad2)
- LED17 pad 1: VCC -> Net-(C23-Pad2)
- LED18 pad 1: VCC -> Net-(C24-Pad2)
- LED19 pad 1: VCC -> Net-(C26-Pad1)
- LED2 pad 1: VCC -> Net-(C8-Pad1)
- LED20 pad 1: VCC -> Net-(C26-Pad2)
- LED21 pad 1: VCC -> Net-(C27-Pad2)
- LED22 pad 1: VCC -> Net-(C28-Pad2)
- LED23 pad 1: VCC -> Net-(C29-Pad2)
- LED24 pad 1: VCC -> Net-(C30-Pad2)
- LED25 pad 1: VCC -> Net-(C31-Pad2)
- LED26 pad 1: VCC -> Net-(C33-Pad1)
- LED27 pad 1: VCC -> Net-(C33-Pad2)
- LED28 pad 1: VCC -> Net-(C34-Pad2)
- LED29 pad 1: VCC -> Net-(C35-Pad2)
- LED3 pad 1: VCC -> Net-(C10-Pad2)
- LED30 pad 1: VCC -> Net-(C36-Pad2)
- LED31 pad 1: VCC -> Net-(C37-Pad2)
- LED4 pad 1: VCC -> Net-(C10-Pad1)
- LED5 pad 1: VCC -> Net-(C12-Pad1)
- LED6 pad 1: VCC -> Net-(C12-Pad2)
- LED7 pad 1: VCC -> Net-(C13-Pad2)
- LED8 pad 1: VCC -> Net-(C14-Pad2)
- LED9 pad 1: VCC -> Net-(C15-Pad2)
- U1 pad 1: Net-(U1-Pad1) -> D-
- U1 pad 2: SERIAL -> GND
- U1 pad 5: Net-(U1-Pad5) -> VBUS
- U1 pad 6: Net-(U1-Pad6) -> D+
Routing:
- net COL0: track 0.00 -> 57.3 mm, vias 0 -> 4
- net Net-(H2-Pad1): track 17.3 -> 0.00 mm
- net Net-(H1-Pad1): track 16.8 -> 0.00 mm

Commit message: Create reversible Cystal footprint
Parts:
- C1, C10, C11, C15, C16, C17, C18, C19, C2, C20, C21, C22, C23, C24, C25, C26, C27, C28, C29, C3, C30, C31, C32, C33, C34, C35, C36, C37, C38, C4, C5, C6, C7, C8, C9: footprint Capacitor_SMD:C_0805_2012Metric -> reversible-kicad-footprints:C-0805_2012Metric
- C12, C13, C14: footprint Capacitor_SMD:C_0805_2012Metric -> reversible-kicad-footprints:C-0805_2012Metric; moved to F.Cu
- D1, D2: footprint Diode_SMD:D_SOD-123 -> reversible-kicad-footprints:D_SOD-123; moved to F.Cu
- D10, D11, D12, D13, D14, D15, D16, D17, D18, D19, D20, D21, D22, D23, D24, D25, D26, D27, D3, D4, D5, D6, D7, D8, D9: footprint Diode_SMD:D_SOD-123 -> reversible-kicad-footprints:D_SOD-123
- F1: footprint Fuse:Fuse_1206_3216Metric -> reversible-kicad-footprints:Fuse_1206_3216Metric
- J2: footprint Connector_USB:USB_C_Receptacle_HRO_TYPE-C-31-M-12 -> reversible-kicad-footprints:HRO-TYPE-C-31-M-12-HandSoldering-NoSBU
- LED1, LED2, LED3, LED4: footprint kbd:YS-SK6812MINI-E -> reversible-kicad-footprints:SK6812Mini-E
- LED10, LED11, LED12, LED13, LED14, LED15, LED16, LED17, LED18, LED19, LED20, LED21, LED22, LED23, LED24, LED25, LED26, LED27, LED28, LED29, LED30, LED31, LED8, LED9: footprint kbd:YS-SK6812MINI-E -> reversible-kicad-footprints:MX-1U-SK6812Mini-E
- LED5, LED6, LED7: footprint kbd:YS-SK6812MINI-E -> reversible-kicad-footprints:MX-1U-SK6812Mini-E; moved to F.Cu
- R1, R2, R3, R4, R5, R6: footprint Resistor_SMD:R_0805_2012Metric -> reversible-kicad-footprints:R-0805_2012Metric
- SW1, SW10, SW11, SW12, SW13, SW14, SW15, SW16, SW17, SW18, SW19, SW2, SW20, SW22, SW23, SW24, SW25, SW26, SW27, SW3, SW4, SW5, SW6, SW7, SW8, SW9: footprint kbd:CherryMX_Hotswap -> reversible-kicad-footprints:MX-1U-Hotswap
- SW21: footprint Keebio-Parts:RotaryEncoder_Alps_EC11E-Switch_Vertical_H20mm -> reversible-kicad-footprints:MX-1U-EC11_Switch
- SW28: footprint random-keyboard-parts:SKQG-1155865 -> reversible-kicad-footprints:SMD_Push
- U1: footprint Package_TO_SOT_SMD:SOT-23-6 -> reversible-kicad-footprints:SOT-23-6
- Y1: footprint Crystal:Crystal_SMD_3225-4Pin_3.2x2.5mm_HandSoldering -> intositeme:Reversible-Crystal_SMD_3225-4pin_3.2x2.5mm
- moved C12 416.0 mm to (516.6, 80.7), turned to 0 degrees
- moved C13 382.8 mm to (500.8, 97.4), turned to 0 degrees
- moved D2 375.3 mm to (491.3, 99.9), turned to 0 degrees
- moved C14 338.1 mm to (469.1, 128.7), turned to 0 degrees
- moved LED6 332.1 mm to (458.3, 50.4), turned to 0 degrees
- moved LED7 252.9 mm to (391.8, 111.0), turned to 0 degrees
- moved LED30 204.7 mm to (310.9, 137.2)
- moved R5 180.8 mm to (525.6, 68.2)
- moved LED3 180.6 mm to (357.8, 164.1)
- moved LED4 161.1 mm to (346.8, 164.1)
- moved Y1 159.1 mm to (367.8, 192.0)
- moved ISP1 159.0 mm to (521.1, 62.9)
- moved J1 149.5 mm to (514.0, 62.9)
- moved R3 142.3 mm to (522.4, 71.7)
- moved U2 137.1 mm to (489.9, 88.0)
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Connections:
- C10 pad 1: Net-(C10-Pad1) -> VBUS
- C10 pad 2: Net-(C10-Pad2) -> GND
- C11 pad 2: Net-(C10-Pad1) -> GND
- C12 pad 1: Net-(C12-Pad1) -> VBUS
- C12 pad 2: Net-(C12-Pad2) -> GND
- C13 pad 1: Net-(C12-Pad2) -> VBUS
- C13 pad 2: Net-(C13-Pad2) -> GND
- C14 pad 1: Net-(C13-Pad2) -> VBUS
- C14 pad 2: Net-(C14-Pad2) -> GND
- C15 pad 1: Net-(C14-Pad2) -> VBUS
- C15 pad 2: Net-(C15-Pad2) -> GND
- C16 pad 1: Net-(C15-Pad2) -> VBUS
- C16 pad 2: Net-(C16-Pad2) -> GND
- C17 pad 1: Net-(C16-Pad2) -> VBUS
- C17 pad 2: Net-(C17-Pad2) -> GND
- C18 pad 1: Net-(C17-Pad2) -> VBUS
- C18 pad 2: VBUS -> GND
- C19 pad 1: Net-(C19-Pad1) -> VBUS
- C19 pad 2: Net-(C19-Pad2) -> GND
- C20 pad 1: Net-(C19-Pad2) -> VBUS
- C20 pad 2: Net-(C20-Pad2) -> GND
- C21 pad 1: Net-(C20-Pad2) -> VBUS
- C21 pad 2: Net-(C21-Pad2) -> GND
- C22 pad 1: Net-(C21-Pad2) -> VBUS
- C22 pad 2: Net-(C22-Pad2) -> GND
- C23 pad 1: Net-(C22-Pad2) -> VBUS
- C23 pad 2: Net-(C23-Pad2) -> GND
- C24 pad 1: Net-(C23-Pad2) -> VBUS
- C24 pad 2: Net-(C24-Pad2) -> GND
- C25 pad 1: Net-(C24-Pad2) -> VBUS
- C25 pad 2: VBUS -> GND
- C26 pad 1: Net-(C26-Pad1) -> VBUS
- C26 pad 2: Net-(C26-Pad2) -> GND
- C27 pad 1: Net-(C26-Pad2) -> VBUS
- C27 pad 2: Net-(C27-Pad2) -> GND
- C28 pad 1: Net-(C27-Pad2) -> VBUS
- C28 pad 2: Net-(C28-Pad2) -> GND
- C29 pad 1: Net-(C28-Pad2) -> VBUS
- C29 pad 2: Net-(C29-Pad2) -> GND
- C30 pad 1: Net-(C29-Pad2) -> VBUS
- C30 pad 2: Net-(C30-Pad2) -> GND
- C31 pad 1: Net-(C30-Pad2) -> VBUS
- C31 pad 2: Net-(C31-Pad2) -> GND
- C32 pad 1: Net-(C31-Pad2) -> VBUS
- C32 pad 2: VBUS -> GND
- C33 pad 1: Net-(C33-Pad1) -> VBUS
- C33 pad 2: Net-(C33-Pad2) -> GND
- C34 pad 1: Net-(C33-Pad2) -> VBUS
- C34 pad 2: Net-(C34-Pad2) -> GND
- C35 pad 1: Net-(C34-Pad2) -> VBUS
- C35 pad 2: Net-(C35-Pad2) -> GND
- C36 pad 1: Net-(C35-Pad2) -> VBUS
- C36 pad 2: Net-(C36-Pad2) -> GND
- C37 pad 1: Net-(C36-Pad2) -> VBUS
- C37 pad 2: Net-(C37-Pad2) -> GND
- C38 pad 1: Net-(C37-Pad2) -> VBUS
- C38 pad 2: VBUS -> GND
- C8 pad 1: Net-(C8-Pad1) -> VBUS
- C8 pad 2: Net-(C8-Pad2) -> GND
- C9 pad 1: Net-(C10-Pad2) -> VBUS
- C9 pad 2: Net-(C8-Pad1) -> GND
- LED1 pad 1: Net-(C8-Pad2) -> VBUS
- LED10 pad 1: Net-(C16-Pad2) -> VBUS
- LED11 pad 1: Net-(C17-Pad2) -> VBUS
- LED12 pad 1: Net-(C19-Pad1) -> VBUS
- LED13 pad 1: Net-(C19-Pad2) -> VBUS
- LED14 pad 1: Net-(C20-Pad2) -> VBUS
- LED15 pad 1: Net-(C21-Pad2) -> VBUS
- LED16 pad 1: Net-(C22-Pad2) -> VBUS
- LED17 pad 1: Net-(C23-Pad2) -> VBUS
- LED18 pad 1: Net-(C24-Pad2) -> VBUS
- LED19 pad 1: Net-(C26-Pad1) -> VBUS
- LED2 pad 1: Net-(C8-Pad1) -> VBUS
- LED20 pad 1: Net-(C26-Pad2) -> VBUS
- LED21 pad 1: Net-(C27-Pad2) -> VBUS
- LED22 pad 1: Net-(C28-Pad2) -> VBUS
- LED23 pad 1: Net-(C29-Pad2) -> VBUS
- LED24 pad 1: Net-(C30-Pad2) -> VBUS
- LED25 pad 1: Net-(C31-Pad2) -> VBUS
- LED26 pad 1: Net-(C33-Pad1) -> VBUS
- LED27 pad 1: Net-(C33-Pad2) -> VBUS
- LED28 pad 1: Net-(C34-Pad2) -> VBUS
- LED29 pad 1: Net-(C35-Pad2) -> VBUS
- LED3 pad 1: Net-(C10-Pad2) -> VBUS
- LED30 pad 1: Net-(C36-Pad2) -> VBUS
- LED31 pad 1: Net-(C37-Pad2) -> VBUS
- LED4 pad 1: Net-(C10-Pad1) -> GND
- LED4 pad 3: GND -> VBUS
- LED5 pad 1: Net-(C12-Pad1) -> VBUS
- LED6 pad 1: Net-(C12-Pad2) -> VBUS
- LED7 pad 1: Net-(C13-Pad2) -> VBUS
- LED8 pad 1: Net-(C14-Pad2) -> VBUS
- LED9 pad 1: Net-(C15-Pad2) -> VBUS
Routing:
- net COL0: track 57.3 -> 0.00 mm, vias 4 -> 0
Other:
- board size 3.6 x 3.1 mm -> 152.4 x 88.1 mm

Commit message: Layout components
Parts:
- removed the C10 at (444.5, 152.0)
- removed the C12 at (516.6, 80.7)
- removed the C13 at (500.8, 97.4)
- removed the C15 at (500.8, 94.5)
- removed the C17 at (489.3, 108.9)
- removed the C19 at (456.0, 142.8)
- removed the C20 at (521.0, 74.8)
- removed C22, C24, C26, C27, C29, C31, C33, C35, C37: 0.1uF, reversible-kicad-footprints:C-0805_2012Metric
- removed the C8 at (484.9, 111.9)
- removed the J2 at (342.9, 204.8)
- removed REF**: Layout, intositeme:Layout
- removed the SW28 at (302.4, 200.0)
- added H1: MountingHole, kbd:M2_HOLE_v3, F.Cu at (116.7, 69.1)
- added H2: MountingHole, kbd:M2_HOLE_v3, F.Cu at (211.9, 69.1)
- added H3: MountingHole, kbd:M2_HOLE_v3, F.Cu at (173.8, 88.1)
- added H4: MountingHole, kbd:M2_HOLE_v3, F.Cu at (116.7, 107.2)
- added H5: MountingHole, kbd:M2_HOLE_v3, F.Cu at (202.4, 107.2)
- added J1: USB_C_Receptacle_USB2.0, reversible-kicad-footprints:HRO-TYPE-C-31-M-12-HandSoldering-NoSBU, F.Cu at (216.4, 47.8)
- added SW22: SW_PUSH, reversible-kicad-footprints:SMD_Push, F.Cu at (246.9, 74.7)
- LED25: footprint reversible-kicad-footprints:MX-1U-SK6812Mini-E -> reversible-kicad-footprints:SK6812Mini-E
- moved LED12 412.7 mm to (107.2, 78.6), turned to 180 degrees
- moved D15 405.8 mm to (107.2, 106.2), turned to 180 degrees
- moved C19 399.1 mm to (119.4, 113.3), turned to 270 degrees
- moved D8 392.9 mm to (107.2, 86.9), turned to 180 degrees
- moved D9 391.6 mm to (126.0, 86.9), turned to 180 degrees
- moved C16 378.8 mm to (138.2, 94.5), turned to 270 degrees
- moved LED13 366.7 mm to (126.2, 78.6), turned to 180 degrees
- moved D2 366.2 mm to (126.5, 68.1), turned to 180 degrees
- moved D24 364.0 mm to (145.3, 125.0), turned to 180 degrees
- moved D3 360.9 mm to (145.3, 68.1), turned to 180 degrees
- moved C12 359.1 mm to (138.2, 75.2), turned to 270 degrees
- moved C20 354.9 mm to (157.5, 113.3), turned to 270 degrees
- moved LED20 347.5 mm to (126.2, 97.6), turned to 180 degrees
- moved D25 345.3 mm to (164.6, 125.0), turned to 180 degrees
- moved C9 338.9 mm to (138.2, 55.9), turned to 270 degrees
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- renumbered C16 to C10, C18 to C11, C21 to C12, C23 to C13, C25 to C14, C7 to C15, C28 to C16, C30 to C17, C32 to C18, C34 to C19, C36 to C20, C38 to C21, C9 to C7, C11 to C8, C14 to C9, J1 to J2, SW21 to SW15, SW15 to SW16, SW16 to SW17, SW17 to SW18, SW18 to SW19, SW19 to SW20, SW20 to SW21, SW22 to SW23, SW23 to SW24, SW24 to SW25, SW25 to SW26, SW26 to SW27, SW27 to SW28
Routing:
- net GND: track 0.00 -> 33.2 mm
- net VBUS: track 0.00 -> 13.9 mm
- net D+: track 0.00 -> 13.3 mm
- net D-: track 0.00 -> 12.0 mm
- net Net-(J1-PadB5): track 0.00 -> 4.25 mm
- net Net-(J1-PadA5): track 0.00 -> 4.01 mm
Other:
- board size 152.4 x 88.1 mm -> 166.2 x 88.1 mm

Commit message: Adding trace
Parts:
- moved R6 2.90 mm to (241.6, 90.7), turned to 180 degrees
- moved C15 1.45 mm to (245.4, 109.2), turned to 180 degrees
- turned C3 to 0 degrees
Routing:
- net ROW0: track 0.00 -> 101.1 mm
- net D+: track 13.3 -> 94.1 mm
- net D-: track 12.0 -> 78.6 mm
- net Net-(LED1-Pad2): track 0.00 -> 66.1 mm, vias 0 -> 2
- net Net-(LED2-Pad4): track 0.00 -> 57.2 mm, vias 0 -> 1
- net Net-(LED1-Pad4): track 0.00 -> 54.6 mm, vias 0 -> 1
- net Net-(LED10-Pad2): track 0.00 -> 53.9 mm
- net LED: track 0.00 -> 43.3 mm
- net Net-(LED3-Pad4): track 0.00 -> 39.7 mm
- net +5V: track 0.00 -> 30.3 mm, vias 0 -> 1
- net Net-(LED12-Pad2): track 0.00 -> 28.8 mm
- net Net-(LED17-Pad4): track 0.00 -> 28.2 mm, vias 0 -> 1
- net Net-(LED11-Pad2): track 0.00 -> 28.1 mm
- net Net-(LED8-Pad2): track 0.00 -> 28.0 mm
- net Net-(LED10-Pad4): track 0.00 -> 28.0 mm
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
Commit message: Done routing.
Parts:
- LED10, LED11, LED19, LED20, LED21, LED22, LED23, LED24, LED5, LED6, LED7, LED8, LED9: moved to B.Cu
- moved R3 47.7 mm to (246.6, 75.8)
- moved ISP1 21.9 mm to (229.6, 119.4), turned to 180 degrees
- moved C3 16.7 mm to (241.6, 94.3), turned to 270 degrees
- moved C2 11.0 mm to (254.3, 84.6)
- moved SW22 7.64 mm to (254.0, 77.5)
- moved R6 6.89 mm to (244.6, 84.5), turned to 90 degrees
- moved C4 6.51 mm to (257.5, 107.4), turned to 0 degrees
- moved J2 4.55 mm to (253.6, 69.8)
- moved C6 4.02 mm to (240.8, 104.7)
- moved Y1 4.02 mm to (250.7, 84.6), turned to 0 degrees
- moved C5 3.95 mm to (254.2, 87.6)
- moved C1 3.54 mm to (247.1, 84.6), turned to 270 degrees
- moved C15 3.47 mm to (248.7, 110.0)
- moved U2 3.31 mm to (250.2, 98.8)
- moved J1 2.38 mm to (216.4, 45.4)
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Connections:
- C7 pad 1: VBUS -> GND
- C7 pad 2: GND -> VBUS
- C8 pad 1: VBUS -> GND
- C8 pad 2: GND -> VBUS
- ISP1 pad 1: MISO -> COL0
- ISP1 pad 2: Net-(ISP1-Pad2) -> VBUS
- ISP1 pad 3: SCK -> COL2
- ISP1 pad 4: MOSI -> COL1
- J2 pad 2: VBUS -> +5V
- LED16 pad 2: Net-(LED15-Pad4) -> Net-(LED16-Pad2)
- LED18 pad 2: Net-(LED17-Pad4) -> Net-(LED18-Pad2)
- LED18 pad 4: Net-(LED11-Pad2) -> Net-(LED18-Pad4)
- LED19 pad 2: Net-(LED19-Pad2) -> Net-(LED1-Pad4)
- LED19 pad 4: Net-(LED12-Pad2) -> Net-(LED19-Pad4)
- LED2 pad 2: Net-(LED1-Pad4) -> Net-(LED2-Pad2)
- LED20 pad 4: Net-(LED19-Pad2) -> Net-(LED1-Pad2)
- LED25 pad 2: Net-(LED25-Pad2) -> Net-(LED18-Pad4)
- LED26 pad 2: Net-(LED26-Pad2) -> Net-(LED19-Pad4)
- LED28 pad 4: Net-(LED28-Pad4) -> Net-(LED2-Pad2)
- LED29 pad 2: Net-(LED28-Pad4) -> Net-(LED2-Pad4)
- LED3 pad 2: Net-(LED2-Pad4) -> Net-(LED15-Pad4)
- LED3 pad 3: GND -> Net-(LED3-Pad3)
- LED3 pad 4: Net-(LED3-Pad4) -> Net-(LED16-Pad2)
- LED31 pad 4: Net-(LED25-Pad2) -> LED
- LED4 pad 1: GND -> VBUS
- LED4 pad 2: Net-(LED3-Pad4) -> Net-(LED17-Pad4)
- LED4 pad 3: VBUS -> GND
- LED4 pad 4: LED -> Net-(LED18-Pad2)
- LED5 pad 4: Net-(LED1-Pad2) -> Net-(LED12-Pad2)
- SW13 pad 1: Net-(SW13-Pad1) -> COL5
- SW14 pad 1: Net-(SW14-Pad1) -> COL6
- SW15 pad S2: Net-(SW14-Pad1) -> COL6
- SW21 pad 1: Net-(SW13-Pad1) -> COL5
- SW28 pad 1: Net-(SW13-Pad1) -> COL5
- SW6 pad 1: Net-(SW13-Pad1) -> COL5
- SW7 pad 1: Net-(SW14-Pad1) -> COL6
- U2 pad 10: MOSI -> COL1
- U2 pad 11: MISO -> COL0
- U2 pad 18: ENC0 -> Net-(U2-Pad18)
- U2 pad 19: ENC1 -> Net-(U2-Pad19)
- U2 pad 22: LED -> Net-(U2-Pad22)
- U2 pad 26: ROW2 -> ROW0
- U2 pad 27: ROW1 -> COL6
- U2 pad 28: ROW0 -> ROW1
- U2 pad 29: COL6 -> ROW2
- U2 pad 30: COL5 -> Net-(U2-Pad30)
- U2 pad 31: COL4 -> Net-(U2-Pad31)
- U2 pad 32: COL3 -> Net-(U2-Pad32)
- U2 pad 36: COL2 -> Net-(U2-Pad36)
- U2 pad 37: COL1 -> Net-(U2-Pad37)
- U2 pad 38: COL0 -> COL5
- U2 pad 39: Net-(U2-Pad39) -> ENC1
- U2 pad 40: Net-(U2-Pad40) -> ENC0
- U2 pad 41: Net-(U2-Pad41) -> COL4
- U2 pad 42: Net-(U2-Pad42) -> LED
- U2 pad 8: Net-(U2-Pad8) -> COL3
- U2 pad 9: SCK -> COL2
Routing:
- net GND: track 54.2 -> 807.5 mm, vias 1 -> 12
- net VBUS: track 13.9 -> 665.5 mm, vias 0 -> 11
- net COL0: track 0.00 -> 208.8 mm, vias 0 -> 6
- net COL2: track 0.00 -> 199.7 mm, vias 0 -> 5
- net COL1: track 0.00 -> 184.8 mm, vias 0 -> 3
- net ROW3: track 0.00 -> 170.5 mm, vias 0 -> 1
- net ROW2: track 0.00 -> 159.6 mm, vias 0 -> 3
- net COL3: track 0.00 -> 151.1 mm, vias 0 -> 4
- net ROW1: track 0.00 -> 149.7 mm, vias 0 -> 1
- net COL4: track 0.00 -> 123.8 mm, vias 0 -> 1
- net +5V: track 30.3 -> 125.2 mm, vias 1 -> 7
- net COL5: track 0.00 -> 92.9 mm
- net RESET: track 0.00 -> 76.4 mm, vias 0 -> 1
- net ROW0: track 101.1 -> 166.9 mm, vias 0 -> 2
- net Net-(LED1-Pad2): track 66.1 -> 3.64 mm, vias 2 -> 0
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Other:
- board size 166.2 x 88.1 mm -> 164.3 x 81 mm
