File: kb-split/kb-split.kicad_pcb (KiCad board)
At the start: 2 copper layers, 164.3 x 81 mm, 125 parts, among them J1 USB_C_Receptacle_USB2.0, J2 Conn_01x03_Male, SW1 SW_PUSH, SW10 SW_PUSH, SW11 SW_PUSH, SW12 SW_PUSH, SW13 SW_PUSH, SW14 SW_PUSH, SW15 Rotary_Encoder_Switch, SW16 SW_PUSH, SW17 SW_PUSH, SW18 SW_PUSH, SW19 SW_PUSH, SW2 SW_PUSH, SW20 SW_PUSH, SW21 SW_PUSH, SW22 SW_PUSH, SW23 SW_PUSH, SW24 SW_PUSH, SW25 SW_PUSH, SW26 SW_PUSH, SW27 SW_PUSH, SW28 SW_PUSH, SW3 SW_PUSH, SW4 SW_PUSH, SW5 SW_PUSH, SW6 SW_PUSH, SW7 SW_PUSH, SW8 SW_PUSH, SW9 SW_PUSH, U1 SRV05-4, U2 ATmega32U4-AU, Y1 Crystal_GND24_Small

Commit message: Rev 1. Sent to manufacture. Added ground fills
Routing:
- added copper zone on B.Cu, net GND
- added copper zone on F.Cu, net GND
Other:
- board text added: "intosite rev 1"
Changed lines of the file:
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@@
   (general
     (thickness 1.6)
-    (drawings 12)
+    (drawings 14)
     (tracks 1233)
     (zones 0)
@@
     (visible_elements FFFFFFFF)
     (pcbplotparams
-      (layerselection 0x010fc_ffffffff)
+      (layerselection 0x010f0_ffffffff)
       (usegerberextensions false)
       (usegerberattributes true)
@@
       (drillshape 0)
       (scaleselection 1)
-      (outputdirectory ""))
+      (outputdirectory "gerbers/"))
   )
   (net 0 "")
@@
     )
   )
+  (gr_text "intosite rev 1" (at 245.999 50.546) (layer B.SilkS)
+    (effects (font (size 1 1) (thickness 0.15)) (justify mirror))
+  )
+  (gr_text "intosite rev 1" (at 246.126 50.546) (layer F.SilkS)
+    (effects (font (size 1 1) (thickness 0.15)))
+  )
   (gr_line (start 256.413 55.626) (end 256.413 58.674) (layer Edge.Cuts) (width 0.1))
   (gr_line (start 245.745 55.626) (end 256.413 55.626) (layer Edge.Cuts) (width 0.1))
@@
   (segment (start 226.568 76.708) (end 226.568 74.93) (width 0.254) (layer F.Cu) (net 94))
   (segment (start 226.568 74.93) (end 226.314 74.676) (width 0.254) (layer F.Cu) (net 94))
+  (zone (net 41) (net_name GND) (layer B.Cu) (hatch edge 0.508)
+    (connect_pads (clearance 0.508))
+    (min_thickness 0.254)
+    (fill yes (arc_segments 32) (thermal_gap 0.508) (thermal_bridge_width 0.508))
+    (polygon
+      (pts
+        (xy 264.668 46.228) (xy 263.525 113.665) (xy 222.504 131.572) (xy 94.869 130.048) (xy 94.488 45.974)
+      )
+    )
+  )
+  (zone (net 41) (net_name GND) (layer F.Cu) (hatch edge 0.508)
+    (connect_pads (clearance 0.508))
+    (min_thickness 0.254)
+    (fill yes (arc_segments 32) (thermal_gap 0.508) (thermal_bridge_width 0.508))
+    (polygon
+      (pts
+        (xy 92.837 44.323) (xy 265.938 44.323) (xy 268.859 132.842) (xy 93.345 132.334) (xy 92.837 44.323)
+        (xy 92.71 44.323) (xy 99.06 42.418)
+      )
+    )
+  )
 )

Commit message: Added trs and fix gerbers export
Parts:
- removed C20, C21: 0.1uF, reversible-kicad-footprints:C-0805_2012Metric
- added J3: AudioPlug3, reversible-kicad-footprints:PJ-3136-B, F.Cu at (259.6, 64.0)
Routing:
- net SERIAL: track 32.6 -> 45.0 mm
- net +5V: track 125.2 -> 136.7 mm
- net GND: track 807.5 -> 818.9 mm
